File: hardware/kicad/Koken-KeyBox.kicad_sch (KiCad schematic)
At the start: 10 parts, among them J1 Jack-DC, J2 LED, J3 Servo

Commit message: コネクタをXHに、電源用コネクタをType-Cに変更
Parts:
- removed J1: Jack-DC, Connector_BarrelJack:BarrelJack_Horizontal, symbol Connector:Jack-DC
- added J4: USB_C_Receptacle_PowerOnly_6P, Connector_USB:USB_C_Receptacle_GCT_USB4125-xx-x_6P_TopMnt_Horizontal, symbol Connector:USB_C_Receptacle_PowerOnly_6P
- added R1, R2: 5.1k, Resistor_SMD:R_0603_1608Metric_Pad0.98x0.95mm_HandSolder, symbol Device:R
- C1, C2: footprint Capacitor_THT:CP_Radial_D5.0mm_P2.50mm -> Capacitor_SMD:C_0603_1608Metric_Pad1.08x0.95mm_HandSolder
- J2, J3: footprint MyLibrary:ZH_3P_Side -> Connector_JST:JST_XH_S3B-XH-A_1x03_P2.50mm_Horizontal
Connections:
- net +5V: now also J4.A9 (VBUS), J4.B9 (VBUS)
- net GND: now also J2.1 (Pin_1), U1.20 (GND), U1.25 (GND), U1.39 (GND), J4.A12 (GND), J4.B12 (GND), J4.S1 (SHIELD), R1.2, R2.2; no longer J2.3 (Pin_3)
- net LED_Failure: now also J2.3 (Pin_3); no longer J2.1 (Pin_1)
- new net: J4.A5 (CC1), R2.1
- new net: J4.B5 (CC2), R1.1
Other:
- moved on the sheet: C2
